File: Main.brd (EAGLE design)
At the start: 53 x 33 mm, 21 parts, among them IC1 LD117AS33TR

Commit message: Added a cutout region under the antenna so that no ground plane is placed there
Parts:
- ESP8266-03: device esp8266modules:ESP-03 -> esp8266modules:ESP03
Routing:
- added copper zone on layer 1, net N$2
Changed lines of the file:
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@@
 </autorouter>
 <elements>
-<element name="ESP8266-03" library="esp8266modules" package="ESP-03" value="ESP8266" x="34.29" y="22.86"/>
+<element name="ESP8266-03" library="esp8266modules" package="ESP03" value="ESP8266" x="34.29" y="22.86"/>
 <element name="FTDI" library="pinhead" package="1X03" value="" x="45.72" y="17.78" rot="R270"/>
 <element name="POWER" library="pinhead" package="1X02" value="" x="45.72" y="8.89" smashed="yes" rot="R270">
@@
 <wire x1="20" y1="17.78" x2="22.708" y2="17.78" width="0.4064" layer="1"/>
 </signal>
+<signal name="N$2">
+<polygon width="0" layer="1" pour="cutout">
+<vertex x="29.21" y="31.75"/>
+<vertex x="41.275" y="31.75"/>
+<vertex x="41.275" y="28.8925"/>
+<vertex x="29.21" y="28.8925"/>
+</polygon>
+</signal>
 </signals>
